File: pcb/energy-management-driver-175.sch (EAGLE design)
At the start: 49 parts, among them T1 BT138-V, T2 BT138-V, T3 BT138-V, T4 BT138-V, T5 BT138-V, T6 BT138-V, T7 BT138-V, T8 BT138-V

Commit message: updated driver board and add input board
Update driver 175 board to use skun terminal. Also add input board for
hotel asia
Parts:
- removed X1, X2, X3, X4, X5, X6, X7, X8: (no value), con-ptr500:AK300/2
- added JP1, JP3, JP4, JP5, JP6, JP7, JP8, JP9: (no value), pinhead:PINHD-1X1
- added U$1, U$2, U$3, U$4, U$5, U$6, U$7, U$8: CONN-SKUN, bontor:CONN-SKUN
Connections:
- net N$15: now also JP3.1; no longer X2-2.KL
- net N$21: now also JP4.1; no longer X3-2.KL
- net N$27: now also JP5.1; no longer X4-2.KL
- net N$33: now also JP9.1; no longer X5-2.KL
- net N$39: now also JP8.1; no longer X6-2.KL
- net N$45: now also JP7.1; no longer X7-2.KL
- net N$51: now also JP6.1; no longer X8-2.KL
- net N$52: now also U$2.P$1; no longer X2-1.KL
- net N$53: now also U$3.P$1; no longer X3-1.KL
- net N$54: now also U$4.P$1; no longer X4-1.KL
- net N$55: now also U$5.P$1; no longer X8-1.KL
- net N$56: now also U$6.P$1; no longer X7-1.KL
- net N$57: now also U$7.P$1; no longer X6-1.KL
- net N$58: now also U$8.P$1; no longer X5-1.KL
- net N$6: now also JP1.1; no longer X1-2.KL
- net N$9: now also U$1.P$1; no longer X1-1.KL
Other:
- note removed: "Switches"
Changed lines of the file:
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@@
 <part name="C16" library="resistor" deviceset="C-EU" device="C0805" value="C0.1uF"/>
 <part name="JP2" library="pinhead" deviceset="PINHD-2X5" device=""/>
-<part name="X1" library="con-ptr500" deviceset="AK300/2" device=""/>
-<part name="X2" library="con-ptr500" deviceset="AK300/2" device=""/>
-<part name="X3" library="con-ptr500" deviceset="AK300/2" device=""/>
-<part name="X4" library="con-ptr500" deviceset="AK300/2" device=""/>
-<part name="X5" library="con-ptr500" deviceset="AK300/2" device=""/>
-<part name="X6" library="con-ptr500" deviceset="AK300/2" device=""/>
-<part name="X7" library="con-ptr500" deviceset="AK300/2" device=""/>
-<part name="X8" library="con-ptr500" deviceset="AK300/2" device=""/>
 <part name="GND2" library="SparkFun-Aesthetics" deviceset="GND" device=""/>
+<part name="JP1" library="pinhead" deviceset="PINHD-1X1" device=""/>
+<part name="U$1" library="bontor" deviceset="CONN-SKUN" device=""/>
+<part name="U$2" library="bontor" deviceset="CONN-SKUN" device=""/>
+<part name="U$3" library="bontor" deviceset="CONN-SKUN" device=""/>
+<part name="U$4" library="bontor" deviceset="CONN-SKUN" device=""/>
+<part name="U$5" library="bontor" deviceset="CONN-SKUN" device=""/>
+<part name="U$6" library="bontor" deviceset="CONN-SKUN" device=""/>
+<part name="U$7" library="bontor" deviceset="CONN-SKUN" device=""/>
+<part name="U$8" library="bontor" deviceset="CONN-SKUN" device=""/>
+<part name="JP3" library="pinhead" deviceset="PINHD-1X1" device=""/>
+<part name="JP4" library="pinhead" deviceset="PINHD-1X1" device=""/>
+<part name="JP5" library="pinhead" deviceset="PINHD-1X1" device=""/>
+<part name="JP6" library="pinhead" deviceset="PINHD-1X1" device=""/>
+<part name="JP7" library="pinhead" deviceset="PINHD-1X1" device=""/>
+<part name="JP8" library="pinhead" deviceset="PINHD-1X1" device=""/>
+<part name="JP9" library="pinhead" deviceset="PINHD-1X1" device=""/>
 </parts>
 <sheets>
 <sheet>
 <plain>
-<text x="91.44" y="172.72" size="2.54" layer="98">Switches</text>
 </plain>
 <instances>
@@
 <instance part="C16" gate="G$1" x="160.02" y="30.48"/>
 <instance part="JP2" gate="A" x="241.3" y="172.72"/>
-<instance part="X1" gate="-1" x="76.2" y="167.64"/>
-<instance part="X1" gate="-2" x="76.2" y="137.16"/>
-<instance part="X2" gate="-1" x="76.2" y="124.46"/>
-<instance part="X2" gate="-2" x="76.2" y="93.98"/>
-<instance part="X3" gate="-1" x="76.2" y="83.82"/>
-<instance part="X3" gate="-2" x="76.2" y="53.34"/>
-<instance part="X4" gate="-1" x="76.2" y="40.64"/>
-<instance part="X4" gate="-2" x="76.2" y="10.16"/>
-<instance part="X5" gate="-1" x="172.72" y="167.64"/>
-<instance part="X5" gate="-2" x="172.72" y="137.16"/>
-<instance part="X6" gate="-1" x="172.72" y="124.46"/>
-<instance part="X6" gate="-2" x="172.72" y="93.98"/>
-<instance part="X7" gate="-1" x="172.72" y="83.82"/>
-<instance part="X7" gate="-2" x="172.72" y="53.34"/>
-<instance part="X8" gate="-1" x="172.72" y="40.64"/>
-<instance part="X8" gate="-2" x="172.72" y="10.16"/>
 <instance part="GND2" gate="1" x="254" y="165.1"/>
+<instance part="JP1" gate="G$1" x="88.9" y="137.16"/>
+<instance part="U$1" gate="G$1" x="88.9" y="167.64"/>
+<instance part="U$2" gate="G$1" x="88.9" y="124.46"/>
+<instance part="U$3" gate="G$1" x="88.9" y="83.82"/>
+<instance part="U$4" gate="G$1" x="88.9" y="40.64"/>
+<instance part="U$5" gate="G$1" x="185.42" y="40.64"/>
+<instance part="U$6" gate="G$1" x="185.42" y="83.82"/>
+<instance part="U$7" gate="G$1" x="185.42" y="124.46"/>
+<instance part="U$8" gate="G$1" x="185.42" y="167.64"/>
+<instance part="JP3" gate="G$1" x="88.9" y="93.98"/>
+<instance part="JP4" gate="G$1" x="88.9" y="53.34"/>
+<instance part="JP5" gate="G$1" x="88.9" y="10.16"/>
+<instance part="JP6" gate="G$1" x="185.42" y="10.16"/>
+<instance part="JP7" gate="G$1" x="185.42" y="53.34"/>
+<instance part="JP8" gate="G$1" x="185.42" y="93.98"/>
+<instance part="JP9" gate="G$1" x="185.42" y="137.16"/>
 </instances>
 <busses>
@@
 <wire x1="81.28" y1="137.16" x2="81.28" y2="142.24" width="0.1524" layer="91"/>
 <junction x="81.28" y="142.24"/>
-<pinref part="X1" gate="-2" pin="KL"/>
+<pinref part="JP1" gate="G$1" pin="1"/>
+<wire x1="86.36" y1="137.16" x2="81.28" y2="137.16" width="0.1524" layer="91"/>
 </segment>
 </net>
@@
 <wire x1="81.28" y1="93.98" x2="81.28" y2="99.06" width="0.1524" layer="91"/>
 <junction x="81.28" y="99.06"/>
-<pinref part="X2" gate="-2" pin="KL"/>
+<pinref part="JP3" gate="G$1" pin="1"/>
+<wire x1="86.36" y1="93.98" x2="81.28" y2="93.98" width="0.1524" layer="91"/>
 </segment>
 </net>
@@
 <wire x1="81.28" y1="53.34" x2="81.28" y2="58.42" width="0.1524" layer="91"/>
 <junction x="81.28" y="58.42"/>
-<pinref part="X3" gate="-2" pin="KL"/>
+<pinref part="JP4" gate="G$1" pin="1"/>
+<wire x1="86.36" y1="53.34" x2="81.28" y2="53.34" width="0.1524" layer="91"/>
 </segment>
 </net>
@@
 <wire x1="81.28" y1="10.16" x2="81.28" y2="15.24" width="0.1524" layer="91"/>
 <junction x="81.28" y="15.24"/>
-<pinref part="X4" gate="-2" pin="KL"/>
+<pinref part="JP5" gate="G$1" pin="1"/>
+<wire x1="86.36" y1="10.16" x2="81.28" y2="10.16" width="0.1524" layer="91"/>
 </segment>
 </net>
@@
 <wire x1="177.8" y1="137.16" x2="177.8" y2="142.24" width="0.1524" layer="91"/>
 <junction x="177.8" y="142.24"/>
-<pinref part="X5" gate="-2" pin="KL"/>
+<pinref part="JP9" gate="G$1" pin="1"/>
+<wire x1="182.88" y1="137.16" x2="177.8" y2="137.16" width="0.1524" layer="91"/>
 </segment>
 </net>
@@
 <wire x1="177.8" y1="99.06" x2="177.8" y2="93.98" width="0.1524" layer="91"/>
 <junction x="177.8" y="99.06"/>
-<pinref part="X6" gate="-2" pin="KL"/>
+<pinref part="JP8" gate="G$1" pin="1"/>
+<wire x1="182.88" y1="93.98" x2="177.8" y2="93.98" width="0.1524" layer="91"/>
 </segment>
 </net>
@@
 <wire x1="177.8" y1="58.42" x2="177.8" y2="53.34" width="0.1524" layer="91"/>
 <junction x="177.8" y="58.42"/>
-<pinref part="X7" gate="-2" pin="KL"/>
+<pinref part="JP7" gate="G$1" pin="1"/>
+<wire x1="182.88" y1="53.34" x2="177.8" y2="53.34" width="0.1524" layer="91"/>
 </segment>
 </net>
@@
 <wire x1="177.8" y1="15.24" x2="177.8" y2="10.16" width="0.1524" layer="91"/>
 <junction x="177.8" y="15.24"/>
-<pinref part="X8" gate="-2" pin="KL"/>
+<pinref part="JP6" gate="G$1" pin="1"/>
+<wire x1="182.88" y1="10.16" x2="177.8" y2="10.16" width="0.1524" layer="91"/>
 </segment>
 </net>
@@
 <wire x1="81.28" y1="167.64" x2="81.28" y2="160.02" width="0.1524" layer="91"/>
 <junction x="81.28" y="160.02"/>
-<pinref part="X1" gate="-1" pin="KL"/>
+<pinref part="U$1" gate="G$1" pin="P$1"/>
 </segment>
 </net>
@@
 <wire x1="81.28" y1="116.84" x2="81.28" y2="124.46" width="0.1524" layer="91"/>
 <junction x="81.28" y="116.84"/>
-<pinref part="X2" gate="-1" pin="KL"/>
+<pinref part="U$2" gate="G$1" pin="P$1"/>
 </segment>
 </net>
@@
 <wire x1="81.28" y1="76.2" x2="81.28" y2="83.82" width="0.1524" layer="91"/>
 <junction x="81.28" y="76.2"/>
-<pinref part="X3" gate="-1" pin="KL"/>
+<pinref part="U$3" gate="G$1" pin="P$1"/>
 </segment>
 </net>
@@
 <wire x1="81.28" y1="33.02" x2="81.28" y2="40.64" width="0.1524" layer="91"/>
 <junction x="81.28" y="33.02"/>
-<pinref part="X4" gate="-1" pin="KL"/>
+<pinref part="U$4" gate="G$1" pin="P$1"/>
 </segment>
 </net>
@@
 <wire x1="177.8" y1="40.64" x2="177.8" y2="33.02" width="0.1524" layer="91"/>
 <junction x="177.8" y="33.02"/>
-<pinref part="X8" gate="-1" pin="KL"/>
+<pinref part="U$5" gate="G$1" pin="P$1"/>
 </segment>
 </net>
@@
 <wire x1="177.8" y1="83.82" x2="177.8" y2="76.2" width="0.1524" layer="91"/>
 <junction x="177.8" y="76.2"/>
-<pinref part="X7" gate="-1" pin="KL"/>
+<pinref part="U$6" gate="G$1" pin="P$1"/>
 </segment>
 </net>
@@
 <wire x1="177.8" y1="124.46" x2="177.8" y2="116.84" width="0.1524" layer="91"/>
 <junction x="177.8" y="116.84"/>
-<pinref part="X6" gate="-1" pin="KL"/>
+<pinref part="U$7" gate="G$1" pin="P$1"/>
 </segment>
 </net>
@@
 <wire x1="177.8" y1="160.02" x2="177.8" y2="167.64" width="0.1524" layer="91"/>
 <junction x="177.8" y="160.02"/>
-<pinref part="X5" gate="-1" pin="KL"/>
-</segment>
-</net>
+<pinref part="U$8" gate="G$1" pin="P$1"/>
+</segment>
+</net>
